Commit message: Double robot config, change a lot of stuff, maybe rebase this commit into multiple commits

File: ws_robotermodelierung/src/my_robot_urdf/urdf/my_robot_urdf.urdf (robot description, URDF)
Before this commit: robot my_robot_urdf, 12 links, 11 joints
Links:
- removed link arm_link_1
- removed link arm_link_2
- removed link arm_link_3
- removed link arm_link_4
- removed link arm_link_5
- removed link arm_link_6
- removed link base_link
- removed link eef_jaw_1
- removed link eef_jaw_2
- removed link eef_jaw_3
- removed link eef_jaw_4
- removed link eef_link
Joints:
- removed joint arm_joint_1
- removed joint arm_joint_2
- removed joint arm_joint_3
- removed joint arm_joint_4
- removed joint arm_joint_5
- removed joint arm_joint_6
- removed joint eef_jaw_1_joint_fixed
- removed joint eef_jaw_2_joint_fixed
- removed joint eef_jaw_3_joint_fixed
- removed joint eef_jaw_4_joint_fixed
- removed joint eef_link_fixed

File: ws_robotermodelierung/src/my_robot_urdf_moveit_config/config/gazebo_my_robot_urdf.urdf (robot description, URDF)
Before this commit: robot my_robot_urdf, 13 links, 12 joints
Links:
- removed link world_link
Joints:
- removed joint base_joint
