Commit message: Added suroundings and replaced robots correctly

File: ws_robotermodelierung/src/my_robot_urdf/urdf/arm_coco.xacro (robot description, xacro)
@@ -6,5 +6,5 @@
             <inertial>
                 <origin
-                    xyz="-0.0764021530191945 2.71349348865523E-05 0.0792317455056668"
+                    xyz="-0.0764021530191945 2.71349348865524E-05 0.0792317455056668"
                     rpy="0 0 0" />
                 <mass
@@ -12,8 +12,8 @@
                 <inertia
                     ixx="0.388653917501998"
-                    ixy="3.7351572975921E-18"
+                    ixy="4.55531640481332E-18"
                     ixz="6.82570301647603E-05"
                     iyy="0.347678993710906"
-                    iyz="9.00213723376388E-18"
+                    iyz="9.04140279476641E-18"
                     izz="0.646698533818771" />
             </inertial>
@@ -52,5 +52,5 @@
             <inertial>
                 <origin
-                    xyz="0.0310954578647585 0.134341853376388 0.00332496023117676"
+                    xyz="0.0310954578647585 -0.00332496023117675 0.134341853376388"
                     rpy="0 0 0" />
                 <mass
@@ -58,9 +58,9 @@
                 <inertia
                     ixx="0.316024916828851"
-                    ixy="-0.0129236801369765"
-                    ixz="0.000189061034524889"
-                    iyy="0.500692862333896"
-                    iyz="0.00031691495962207"
-                    izz="0.322997369549128" />
+                    ixy="-0.000189061034524887"
+                    ixz="-0.0129236801369765"
+                    iyy="0.322997369549128"
+                    iyz="-0.000316914959622081"
+                    izz="0.500692862333896" />
             </inertial>
             <visual>
@@ -93,67 +93,9 @@
             <origin
                 xyz="0 0 0.18"
-                rpy="1.5708 0 0" />
+                rpy="0 0 0" />
             <parent
                 link="${prefix}base_link_coco" />
             <child
                 link="${prefix}arm_link_1_coco" />
-            <axis
-                xyz="0 1 0" />
-            <limit
-                lower="-3.1416"
-                upper="3.1416"
-                effort="0"
-                velocity="0" />
-        </joint>
-        <link
-            name="${prefix}arm_link_2_coco">
-            <inertial>
-                <origin
-                    xyz="0.0252292801061356 0.315341966336714 0.119016776091288"
-                    rpy="0 0 0" />
-                <mass
-                    value="29.9902849835083" />
-                <inertia
-                    ixx="2.0278918621324"
-                    ixy="-0.156444807181449"
-                    ixz="2.66331568201595E-17"
-                    iyy="0.155884497994694"
-                    iyz="2.4398292141135E-17"
-                    izz="2.1168438189684" />
-            </inertial>
-            <visual>
-                <origin
-                    xyz="0 0 0"
-                    rpy="0 0 0" />
-                <geometry>
-                    <mesh
-                        filename="package://my_robot_urdf/meshes/arm_link_2_coco.STL" />
-                </geometry>
-                <material
-                    name="">
-                    <color
-                        rgba="0.792156862745098 0.819607843137255 0.933333333333333 1" />
-                </material>
-            </visual>
-            <collision>
-                <origin
-                    xyz="0 0 0"
-                    rpy="0 0 0" />
-                <geometry>
-                    <mesh
-                        filename="package://my_robot_urdf/meshes/arm_link_2_coco.STL" />
-                </geometry>
-            </collision>
-        </link>
-        <joint
-            name="${prefix}joint_link_2_coco"
-            type="revolute">
-            <origin
-                xyz="0.14579 0.33595 0.090292"
-                rpy="0 0 0.082805" />
-            <parent
-                link="${prefix}arm_link_1_coco" />
-            <child
-                link="${prefix}arm_link_2_coco" />
             <axis
                 xyz="0 0 1" />
@@ -165,53 +107,53 @@
         </joint>
         <link
-            name="${prefix}arm_link_3_coco">
-            <inertial>
-                <origin
-                    xyz="0.170027563293456 0.0889986484280518 -0.0663605481820072"
-                    rpy="0 0 0" />
-                <mass
-                    value="16.1199771168543" />
-                <inertia
-                    ixx="0.137763861529296"
-                    ixy="-0.0959483935903458"
-                    ixz="-0.0167225971301647"
-                    iyy="0.190812936291584"
-                    iyz="-0.012987856550598"
-                    izz="0.261074961271267" />
-            </inertial>
-            <visual>
-                <origin
-                    xyz="0 0 0"
-                    rpy="0 0 0" />
-                <geometry>
-                    <mesh
-                        filename="package://my_robot_urdf/meshes/arm_link_3_coco.STL" />
-                </geometry>
-                <material
-                    name="">
-                    <color
-                        rgba="0.792156862745098 0.819607843137255 0.933333333333333 1" />
-                </material>
-            </visual>
-            <collision>
-                <origin
-                    xyz="0 0 0"
-                    rpy="0 0 0" />
-                <geometry>
-                    <mesh
-                        filename="package://my_robot_urdf/meshes/arm_link_3_coco.STL" />
-                </geometry>
-            </collision>
-        </link>
-        <joint
-            name="${prefix}joint_link_3_coco"
+            name="${prefix}arm_link_2_coco">
+            <inertial>
+                <origin
+                    xyz="-0.000939286587736787 0.316348210123726 0.119016776091287"
+                    rpy="0 0 0" />
+                <mass
+                    value="29.9902849835083" />
+                <inertia
+                    ixx="2.04087599375796"
+                    ixy="7.61592373322073E-18"
+                    ixz="2.46332916825912E-17"
+                    iyy="0.14290036636914"
+                    iyz="1.17013190501613E-17"
+                    izz="2.11684381896841" />
+            </inertial>
+            <visual>
+                <origin
+                    xyz="0 0 0"
+                    rpy="0 0 0" />
+                <geometry>
+                    <mesh
+                        filename="package://my_robot_urdf/meshes/arm_link_2_coco.STL" />
+                </geometry>
+                <material
+                    name="">
+                    <color
+                        rgba="0.792156862745098 0.819607843137255 0.933333333333333 1" />
+                </material>
+            </visual>
+            <collision>
+                <origin
+                    xyz="0 0 0"
+                    rpy="0 0 0" />
+                <geometry>
+                    <mesh
+                        filename="package://my_robot_urdf/meshes/arm_link_2_coco.STL" />
+                </geometry>
+            </collision>
+        </link>
+        <joint
+            name="${prefix}joint_link_2_coco"
             type="revolute">
             <origin
-                xyz="0.0017779 0.76236 0"
-                rpy="0 0 -0.082805" />
-            <parent
+                xyz="0.14579 -0.090292 0.33595"
+                rpy="1.5708 0 0" />
+            <parent
+                link="${prefix}arm_link_1_coco" />
+            <child
                 link="${prefix}arm_link_2_coco" />
-            <child
-                link="${prefix}arm_link_3_coco" />
             <axis
                 xyz="0 0 1" />
@@ -223,55 +165,55 @@
         </joint>
         <link
-            name="${prefix}arm_link_4_coco">
-            <inertial>
-                <origin
-                    xyz="0.227600947287535 0.0354202245742417 -0.00589018251913133"
-                    rpy="0 0 0" />
-                <mass
-                    value="8.2144132017799" />
-                <inertia
-                    ixx="0.0518416725365333"
-                    ixy="-0.0168710233275404"
-                    ixz="1.62360283324883E-05"
-                    iyy="0.164102263665489"
-                    iyz="1.53545094184089E-06"
-                    izz="0.160372113366996" />
-            </inertial>
-            <visual>
-                <origin
-                    xyz="0 0 0"
-                    rpy="0 0 0" />
-                <geometry>
-                    <mesh
-                        filename="package://my_robot_urdf/meshes/arm_link_4_coco.STL" />
-                </geometry>
-                <material
-                    name="">
-                    <color
-                        rgba="0.792156862745098 0.819607843137255 0.933333333333333 1" />
-                </material>
-            </visual>
-            <collision>
-                <origin
-                    xyz="0 0 0"
-                    rpy="0 0 0" />
-                <geometry>
-                    <mesh
-                        filename="package://my_robot_urdf/meshes/arm_link_4_coco.STL" />
-                </geometry>
-            </collision>
-        </link>
-        <joint
-            name="${prefix}joint_link_4_coco"
+            name="${prefix}arm_link_3_coco">
+            <inertial>
+                <origin
+                    xyz="0.106966394959347 -0.0865335610269826 0.0663605481820073"
+                    rpy="0 0 0" />
+                <mass
+                    value="16.1199771168543" />
+                <inertia
+                    ixx="0.137763861529296"
+                    ixy="0.0959483935903455"
+                    ixz="0.0167225971301647"
+                    iyy="0.190812936291584"
+                    iyz="-0.012987856550598"
+                    izz="0.261074961271267" />
+            </inertial>
+            <visual>
+                <origin
+                    xyz="0 0 0"
+                    rpy="0 0 0" />
+                <geometry>
+                    <mesh
+                        filename="package://my_robot_urdf/meshes/arm_link_3_coco.STL" />
+                </geometry>
+                <material
+                    name="">
+                    <color
+                        rgba="0.792156862745098 0.819607843137255 0.933333333333333 1" />
+                </material>
+            </visual>
+            <collision>
+                <origin
+                    xyz="0 0 0"
+                    rpy="0 0 0" />
+                <geometry>
+                    <mesh
+                        filename="package://my_robot_urdf/meshes/arm_link_3_coco.STL" />
+                </geometry>
+            </collision>
+        </link>
+        <joint
+            name="${prefix}joint_link_3_coco"
             type="revolute">
             <origin
-                xyz="0.34817 0.19918 -0.073652"
-                rpy="0 0 0" />
-            <parent
+                xyz="0.0017779 0.76236 0"
+                rpy="3.1416 0 0" />
+            <parent
+                link="${prefix}arm_link_2_coco" />
+            <child
                 link="${prefix}arm_link_3_coco" />
-            <child
-                link="${prefix}arm_link_4_coco" />
-            <axis
-                xyz="1 0 0" />
+            <axis
+                xyz="0 0 -1" />
             <limit
                 lower="-3.1416"
@@ -281,53 +223,53 @@
         </joint>
         <link
-            name="${prefix}arm_link_5_coco">
-            <inertial>
-                <origin
-                    xyz="0.074010927598714 0.00261570038501091 -0.0027964156486263"
-                    rpy="0 0 0" />
-                <mass
-                    value="1.15468077380916" />
-                <inertia
-                    ixx="0.0024180307299129"
-                    ixy="-7.71125501828711E-06"
-                    ixz="6.55345310597883E-07"
-                    iyy="0.00301389716175276"
-                    iyz="9.01091984498959E-09"
-                    izz="0.00180806969473038" />
-            </inertial>
-            <visual>
-                <origin
-                    xyz="0 0 0"
-                    rpy="0 0 0" />
-                <geometry>
-                    <mesh
-                        filename="package://my_robot_urdf/meshes/arm_link_5_coco.STL" />
-                </geometry>
-                <material
-                    name="">
-                    <color
-                        rgba="0.792156862745098 0.819607843137255 0.933333333333333 1" />
-                </material>
-            </visual>
-            <collision>
-                <origin
-                    xyz="0 0 0"
-                    rpy="0 0 0" />
-                <geometry>
-                    <mesh
-                        filename="package://my_robot_urdf/meshes/arm_link_5_coco.STL" />
-                </geometry>
-            </collision>
-        </link>
-        <joint
-            name="${prefix}joint_link_5_coco"
+            name="${prefix}arm_link_4_coco">
+            <inertial>
+                <origin
+                    xyz="0.00589018251913124 0.0329551371731716 0.164539778953426"
+                    rpy="0 0 0" />
+                <mass
+                    value="8.2144132017799" />
+                <inertia
+                    ixx="0.160372113366996"
+                    ixy="-1.53545094183557E-06"
+                    ixz="-1.62360283324984E-05"
+                    iyy="0.164102263665489"
+                    iyz="-0.0168710233275404"
+                    izz="0.0518416725365331" />
+            </inertial>
+            <visual>
+                <origin
+                    xyz="0 0 0"
+                    rpy="0 0 0" />
+                <geometry>
+                    <mesh
+                        filename="package://my_robot_urdf/meshes/arm_link_4_coco.STL" />
+                </geometry>
+                <material
+                    name="">
+                    <color
+                        rgba="0.792156862745098 0.819607843137255 0.933333333333333 1" />
+                </material>
+            </visual>
+            <collision>
+                <origin
+                    xyz="0 0 0"
+                    rpy="0 0 0" />
+                <geometry>
+                    <mesh
+                        filename="package://my_robot_urdf/meshes/arm_link_4_coco.STL" />
+                </geometry>
+            </collision>
+        </link>
+        <joint
+            name="${prefix}joint_link_4_coco"
             type="revolute">
             <origin
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
File: ws_robotermodelierung/src/my_robot_urdf/urdf/robot.urdf (robot description, URDF)
Before this commit: robot my_robot, 28 links, 27 joints
Links:
- removed link coco_arm_link_1_coco
- removed link coco_arm_link_2_coco
- removed link coco_arm_link_3_coco
- removed link coco_arm_link_4_coco
- removed link coco_arm_link_5_coco
- removed link coco_arm_link_6_coco
- removed link coco_base_link_coco
- removed link coco_eef_link_1_coco
- removed link coco_eef_link_2_coco
- added link centrifuge_1, mass 500.0; collision cylinder length=0.75 radius=0.5; visual cylinder length=0.75 radius=0.5
- added link centrifuge_2, mass 500.0; collision cylinder length=0.75 radius=0.5; visual cylinder length=0.75 radius=0.5
- added link main_workbench_3, mass 1000.0; collision box size=0.8 5 0.75; visual box size=0.8 5 0.75
- link main_workbench: geometry collision box size=15 15 0.1; visual box size=15 15 0.1
- link main_workbench_2: geometry collision box size=0.8 5 0.75; visual box size=0.8 5 0.75
Joints:
- removed joint coco_arm_joint_6_coco
- removed joint coco_base_joint_coco
- removed joint coco_eef_joint_1_fixed_coco
- removed joint coco_eef_joint_2_fixed_coco
- removed joint coco_joint_link_1_coco
- removed joint coco_joint_link_2_coco
- removed joint coco_joint_link_3_coco
- removed joint coco_joint_link_4_coco
- removed joint coco_joint_link_5_coco
- added joint base_to_centrifuge_1_joint: type fixed, parent central_base_link, child centrifuge_1, origin xyz=1.7 1.2 0 rpy=0 0 0
- added joint base_to_centrifuge_2_joint: type fixed, parent central_base_link, child centrifuge_2, origin xyz=-1.7 1.2 0 rpy=0 0 0
- added joint base_to_workbench_3_joint: type fixed, parent central_base_link, child main_workbench_3, origin xyz=-2.2 -2.5 0 rpy=0 0 0
- joint alex_base_joint_alex: origin xyz=0 0 0.1 rpy=0 0 0 -> xyz=-1 0 0.1 rpy=0 0 3.14159265359
- joint base_to_workbench_2_joint: origin xyz=2.5 0 0 rpy=0 0 0 -> xyz=2.2 -2.5 0 rpy=0 0 0
- joint yuzi_base_joint_yuzi: origin xyz=0 2 0.1 rpy=0 0 0 -> xyz=1 0 0.1 rpy=0 0 0

File: ws_robotermodelierung/src/my_robot_urdf/urdf/robot.xacro (robot description, xacro)
@@ -1,20 +1,48 @@
 <?xml version="1.0"?>
 <robot xmlns:xacro="http://www.ros.org/wiki/xacro" name="my_robot">
+    <!-- Constants -->
+    <xacro:property name="PI" value="3.14159265359" />
+    <!-- Include the xacro files for the utilities and the robot arms -->
+    <xacro:include filename="$(find my_robot_urdf)/urdf/centrifuge.xacro" />
     <xacro:include filename="$(find my_robot_urdf)/urdf/workbench.xacro" />
+    <xacro:include filename="$(find my_robot_urdf)/urdf/workbench_ground.xacro" />
     <xacro:include filename="$(find my_robot_urdf)/urdf/arm.xacro" />
-    <xacro:include filename="$(find my_robot_urdf)/urdf/arm_coco.xacro" />
+    <!-- TODO: Include the arm_coco.xacro file -->
+    <!-- <xacro:include filename="$(find my_robot_urdf)/urdf/arm_coco.xacro" /> -->
     <xacro:include filename="$(find my_robot_urdf)/urdf/arm_yuzi.xacro" />
+    <xacro:property name="robot_alex_distance" value="1.8" />
+    <xacro:property name="robot_yuzi_distance" value="1.8" />
+    <xacro:property name="centrifuge_distance_x" value="1.2" />
+    <xacro:property name="centrifuge_distance_y" value="1.2" />
     <!-- Define parameters for workbench 1-->
     <xacro:property name="workbench_height_1" value="0.1" />
-    <xacro:property name="workbench_length_1" value="2" />
-    <xacro:property name="workbench_width_1" value="5" />
+    <xacro:property name="workbench_length_1" value="15" />
+    <xacro:property name="workbench_width_1" value="15" />
     <xacro:property name="workbench_name_1" value="main_workbench" />
-    <xacro:property name="workbench_height_2" value="0.6" />
-    <xacro:property name="workbench_length_2" value="2" />
+    <!-- Define parameters for workbench 2-->
+    <xacro:property name="workbench_height_2" value="0.75" />
+    <xacro:property name="workbench_length_2" value="0.8" />
     <xacro:property name="workbench_width_2" value="5" />
     <xacro:property name="workbench_name_2" value="main_workbench_2" />
-    <!-- Instantiate the workbench 1 as the root link -->
-    <xacro:workbench workbench_name="${workbench_name_1}" workbench_height="${workbench_height_1}" workbench_length="${workbench_length_1}" workbench_width="${workbench_width_1}" />
+    <!-- Define parameters for workbench 3-->
+    <xacro:property name="workbench_height_3" value="0.75" />
+    <xacro:property name="workbench_length_3" value="0.8" />
+    <xacro:property name="workbench_width_3" value="5" />
+    <xacro:property name="workbench_name_3" value="main_workbench_3" />
+    <!-- Define parameters for centrifuge 1-->
+    <xacro:property name="centrifuge_length_1" value ="0.75" />
+    <xacro:property name="centrifuge_diameter_1" value="1" />
+    <xacro:property name="centrifuge_name_1" value="centrifuge_1" />
+    <!-- Define parameters for centrifuge 2-->
+    <xacro:property name="centrifuge_length_2" value ="0.75" />
+    <xacro:property name="centrifuge_diameter_2" value="1" />
+    <xacro:property name="centrifuge_name_2" value="centrifuge_2" />
+    <!-- Instantiate the workbenches as the root link -->
+    <xacro:workbench_ground workbench_name="${workbench_name_1}" workbench_height="${workbench_height_1}" workbench_length="${workbench_length_1}" workbench_width="${workbench_width_1}" />
     <xacro:workbench workbench_name="${workbench_name_2}" workbench_height="${workbench_height_2}" workbench_length="${workbench_length_2}" workbench_width="${workbench_width_2}" />
+    <xacro:workbench workbench_name="${workbench_name_3}" workbench_height="${workbench_height_3}" workbench_length="${workbench_length_3}" workbench_width="${workbench_width_3}" />
+    <!-- Instantiate the centrifuges as the root link -->
+    <xacro:centrifuge centrifuge_name="${centrifuge_name_1}" centrifuge_length="${centrifuge_length_1}" centrifuge_diameter="${centrifuge_diameter_1}" />
+    <xacro:centrifuge centrifuge_name="${centrifuge_name_2}" centrifuge_length="${centrifuge_length_2}" centrifuge_diameter="${centrifuge_diameter_2}" />
     <!-- Main body link (central base link) -->
     <link name="central_base_link">
@@ -30,9 +58,26 @@
         <parent link="central_base_link"/>
         <child link="${workbench_name_2}"/>
-        <origin xyz="${workbench_width_1/2} 0 0" rpy="0 0 0"/>
+        <origin xyz="${(workbench_length_2 / 2) + robot_alex_distance} -${workbench_width_2 / 2} 0" rpy="0 0 0"/>
+    </joint>
+    <joint name="base_to_workbench_3_joint" type="fixed">
+        <parent link="central_base_link"/>
+        <child link="${workbench_name_3}"/>
+        <origin xyz="-${(workbench_length_3 / 2) + robot_yuzi_distance} -${workbench_width_3 / 2} 0" rpy="0 0 0"/>
+    </joint>
+    <!-- Connect each centrifuge to the central base link with a fixed joint -->
+    <joint name="base_to_centrifuge_1_joint" type="fixed">
+        <parent link="central_base_link"/>
+        <child link="${centrifuge_name_1}"/>
+        <origin xyz="${(centrifuge_diameter_1 / 2) + centrifuge_distance_x} ${centrifuge_distance_y} 0" rpy="0 0 0"/>
+    </joint>
+    <joint name="base_to_centrifuge_2_joint" type="fixed">
+        <parent link="central_base_link"/>
+        <child link="${centrifuge_name_2}"/>
+        <origin xyz="-${(centrifuge_diameter_1 / 2) + centrifuge_distance_x} ${centrifuge_distance_y} 0" rpy="0 0 0"/>
     </joint>
     <!-- Instantiate the arms, attaching it to the central base link -->
-    <xacro:arm prefix="alex_" parent_link="central_base_link" xyz="0 0 ${workbench_height_1}" rpy="0 0 0" />
-    <xacro:arm_coco prefix="coco_" parent_link="central_base_link" xyz="0 1 ${workbench_height_1}" rpy="0 0 0" />
-    <xacro:arm_yuzi prefix="yuzi_" parent_link="central_base_link" xyz="0 2 ${workbench_height_1}" rpy="0 0 0" />
+    <xacro:arm prefix="alex_" parent_link="central_base_link" xyz="-1 0 ${workbench_height_1}" rpy="0 0 ${PI}" />
+    <!-- TODO: Instantiate the arm_coco, attaching it to the central base link -->
+    <!-- <xacro:arm_coco prefix="coco_" parent_link="central_base_link" xyz="0 1 ${workbench_height_1}" rpy="0 0 0" /> -->
+    <xacro:arm_yuzi prefix="yuzi_" parent_link="central_base_link" xyz="1 0 ${workbench_height_1}" rpy="0 0 0" />
 </robot>
