Commit message: Added suroundings and replaced robots correctly

File: ws_robotermodelierung/src/my_robot_urdf/urdf/workbench_ground.xacro (robot description, xacro)
@@ -1,5 +1,5 @@
 <?xml version="1.0"?>
 <robot xmlns:xacro="http://www.ros.org/wiki/xacro">
-    <xacro:macro name="workbench" params="workbench_name workbench_height=1.0 workbench_length=2 workbench_width=2">
+    <xacro:macro name="workbench_ground" params="workbench_name workbench_height=1.0 workbench_length=2 workbench_width=2">
         <link name="${workbench_name}">
             <inertial>
@@ -13,6 +13,6 @@
                     <box size="${workbench_length} ${workbench_width} ${workbench_height}"/>
                 </geometry>
-                <material name="rubber_black">
-                    <color rgba="0.05 0.05 0.05 1"/> <!-- Dark grey to mimic black rubber -->
+                <material name="light_grey">
+                    <color rgba="0.7 0.7 0.7 1"/> <!-- White grey color -->
                 </material>
             </visual>

Commit message: Add centrifuge and correct robot model for cocos robot

File: ws_robotermodelierung/src/my_robot_urdf/urdf/arm_coco.xacro (robot description, xacro)
@@ -6,5 +6,5 @@
             <inertial>
                 <origin
-                    xyz="-0.0764021530191945 2.71349348865524E-05 0.0792317455056668"
+                    xyz="-0.0764021530191944 2.71349348865524E-05 0.0792317455056668"
                     rpy="0 0 0" />
                 <mass
@@ -12,8 +12,8 @@
                 <inertia
                     ixx="0.388653917501998"
-                    ixy="4.55531640481332E-18"
+                    ixy="3.75787448655195E-18"
                     ixz="6.82570301647603E-05"
                     iyy="0.347678993710906"
-                    iyz="9.04140279476641E-18"
+                    iyz="8.89625811535709E-18"
                     izz="0.646698533818771" />
             </inertial>
@@ -116,8 +116,8 @@
                 <inertia
                     ixx="2.04087599375796"
-                    ixy="7.61592373322073E-18"
-                    ixz="2.46332916825912E-17"
+                    ixy="6.72038874095361E-18"
+                    ixz="2.43431801579158E-17"
                     iyy="0.14290036636914"
-                    iyz="1.17013190501613E-17"
+                    iyz="1.09136139887468E-17"
                     izz="2.11684381896841" />
             </inertial>
@@ -168,5 +168,5 @@
             <inertial>
                 <origin
-                    xyz="0.106966394959347 -0.0865335610269826 0.0663605481820073"
+                    xyz="-0.106966394959347 0.0865335610269826 0.0663605481820073"
                     rpy="0 0 0" />
                 <mass
@@ -175,7 +175,7 @@
                     ixx="0.137763861529296"
                     ixy="0.0959483935903455"
-                    ixz="0.0167225971301647"
+                    ixz="-0.0167225971301647"
                     iyy="0.190812936291584"
-                    iyz="-0.012987856550598"
+                    iyz="0.012987856550598"
                     izz="0.261074961271267" />
             </inertial>
@@ -209,5 +209,5 @@
             <origin
                 xyz="0.0017779 0.76236 0"
-                rpy="3.1416 0 0" />
+                rpy="3.1416 0 3.1416" />
             <parent
                 link="${prefix}arm_link_2_coco" />
@@ -232,6 +232,6 @@
                 <inertia
                     ixx="0.160372113366996"
-                    ixy="-1.53545094183557E-06"
-                    ixz="-1.62360283324984E-05"
+                    ixy="-1.53545094183617E-06"
+                    ixz="-1.62360283324988E-05"
                     iyy="0.164102263665489"
                     iyz="-0.0168710233275404"
@@ -266,6 +266,6 @@
             type="revolute">
             <origin
-                xyz="0.34817 -0.19918 0.073652"
-                rpy="0 -1.5708 0" />
+                xyz="-0.34817 0.19918 0.073652"
+                rpy="3.1416 -1.5708 3.1416" />
             <parent
                 link="${prefix}arm_link_3_coco" />
@@ -284,5 +284,5 @@
             <inertial>
                 <origin
-                    xyz="0.010949759264604 0.000150612983941256 -0.00279641564862638"
+                    xyz="0.010949759264604 0.000150612983941256 -0.00279641564862637"
                     rpy="0 0 0" />
                 <mass
@@ -400,5 +400,5 @@
             <inertial>
                 <origin
-                    xyz="3.29649640917751E-11 -9.2350714006928E-05 -0.124708296392705"
+                    xyz="3.29649640917751E-11 -9.235071400715E-05 -0.124708296392705"
                     rpy="0 0 0" />
                 <mass
@@ -459,8 +459,8 @@
                 <inertia
                     ixx="0.000149672253524412"
-                    ixy="-4.86614844728464E-21"
-                    ixz="-1.82017122285296E-21"
+                    ixy="-4.9614680881843E-21"
+                    ixz="7.79229232056955E-22"
                     iyy="0.000192557897320206"
-                    iyz="1.30305666194518E-20"
+                    iyz="1.28004734861553E-20"
                     izz="0.00016094527647324" />
             </inertial>

File: ws_robotermodelierung/src/my_robot_urdf/urdf/robot.urdf (robot description, URDF)
Before this commit: robot my_robot, 22 links, 21 joints
Links:
- added link centrifuge_link_1, mass 1.0; collision mesh filename=package://my_robot_urdf/models/centrifuge.dae scale=1 1 1; visual mesh filename=package://my_robot_urdf/models/centrifuge.dae scale=1 1 1
- added link coco_arm_link_1_coco, mass 28.7973325809481; collision mesh filename=package://my_robot_urdf/meshes/arm_link_1_coco.STL; visual mesh filename=package://my_robot_urdf/meshes/arm_link_1_coco.STL
- added link coco_arm_link_2_coco, mass 29.9902849835083; collision mesh filename=package://my_robot_urdf/meshes/arm_link_2_coco.STL; visual mesh filename=package://my_robot_urdf/meshes/arm_link_2_coco.STL
- added link coco_arm_link_3_coco, mass 16.1199771168543; collision mesh filename=package://my_robot_urdf/meshes/arm_link_3_coco.STL; visual mesh filename=package://my_robot_urdf/meshes/arm_link_3_coco.STL
- added link coco_arm_link_4_coco, mass 8.2144132017799; collision mesh filename=package://my_robot_urdf/meshes/arm_link_4_coco.STL; visual mesh filename=package://my_robot_urdf/meshes/arm_link_4_coco.STL
- added link coco_arm_link_5_coco, mass 1.15468077380916; collision mesh filename=package://my_robot_urdf/meshes/arm_link_5_coco.STL; visual mesh filename=package://my_robot_urdf/meshes/arm_link_5_coco.STL
- added link coco_arm_link_6_coco, mass 1.15468077380916; collision mesh filename=package://my_robot_urdf/meshes/arm_link_6_coco.STL; visual mesh filename=package://my_robot_urdf/meshes/arm_link_6_coco.STL
- added link coco_base_link_coco, mass 33.7641312353281; collision mesh filename=package://my_robot_urdf/meshes/base_link_coco.STL; visual mesh filename=package://my_robot_urdf/meshes/base_link_coco.STL
- added link coco_eef_link_1_coco, mass 0.15332063940157; collision mesh filename=package://my_robot_urdf/meshes/eef_link_1_coco.STL; visual mesh filename=package://my_robot_urdf/meshes/eef_link_1_coco.STL
- added link coco_eef_link_2_coco, mass 0.158859300753402; collision mesh filename=package://my_robot_urdf/meshes/eef_link_2_coco.STL; visual mesh filename=package://my_robot_urdf/meshes/eef_link_2_coco.STL
Joints:
- added joint base_to_centrifuge_model_1_joint: type fixed, parent central_base_link, child centrifuge_link_1, origin xyz=1.7 1.2 0.9379 rpy=1.570796326795 0 0
- added joint coco_arm_joint_6_coco: type revolute, parent coco_arm_link_5_coco, child coco_arm_link_6_coco, origin xyz=0.085 0.00067738 -0.0028482 rpy=0 1.5708 0, axis 0 0 -1, limit lower=-3.1416 upper=3.1416 effort=0 velocity=0
- added joint coco_base_joint_coco: type fixed, parent central_base_link, child coco_base_link_coco, origin xyz=0 1 0.1 rpy=0 0 0
- added joint coco_eef_joint_1_fixed_coco: type fixed, parent coco_arm_link_6_coco, child coco_eef_link_1_coco, origin xyz=0.20975 0.00067738 0.085 rpy=-1.5708 0 -1.5708, axis 0 0 0
- added joint coco_eef_joint_2_fixed_coco: type fixed, parent coco_arm_link_6_coco, child coco_eef_link_2_coco, origin xyz=-0.13985 0.00067738 0.085 rpy=-1.5708 0 1.5708, axis 0 0 0
- added joint coco_joint_link_1_coco: type revolute, parent coco_base_link_coco, child coco_arm_link_1_coco, origin xyz=0 0 0.18 rpy=0 0 0, axis 0 0 1, limit lower=-3.1416 upper=3.1416 effort=0 velocity=0
- added joint coco_joint_link_2_coco: type revolute, parent coco_arm_link_1_coco, child coco_arm_link_2_coco, origin xyz=0.14579 -0.090292 0.33595 rpy=1.5708 0 0, axis 0 0 1, limit lower=-3.1416 upper=3.1416 effort=0 velocity=0
- added joint coco_joint_link_3_coco: type revolute, parent coco_arm_link_2_coco, child coco_arm_link_3_coco, origin xyz=0.0017779 0.76236 0 rpy=3.1416 0 3.1416, axis 0 0 -1, limit lower=-3.1416 upper=3.1416 effort=0 velocity=0
- added joint coco_joint_link_4_coco: type revolute, parent coco_arm_link_3_coco, child coco_arm_link_4_coco, origin xyz=-0.34817 0.19918 0.073652 rpy=3.1416 -1.5708 3.1416, axis 0 0 1, limit lower=-3.1416 upper=3.1416 effort=0 velocity=0
- added joint coco_joint_link_5_coco: type revolute, parent coco_arm_link_4_coco, child coco_arm_link_5_coco, origin xyz=0 0.0656 0.50466 rpy=3.1416 -1.5708 0, axis 0 0 1, limit lower=-3.1416 upper=3.1416 effort=0 velocity=0

File: ws_robotermodelierung/src/my_robot_urdf/urdf/robot.xacro (robot description, xacro)
@@ -8,6 +8,7 @@
     <xacro:include filename="$(find my_robot_urdf)/urdf/workbench_ground.xacro" />
     <xacro:include filename="$(find my_robot_urdf)/urdf/arm.xacro" />
+    <xacro:include filename="$(find my_robot_urdf)/urdf/centrifuge_model.xacro" />
     <!-- TODO: Include the arm_coco.xacro file -->
-    <!-- <xacro:include filename="$(find my_robot_urdf)/urdf/arm_coco.xacro" /> -->
+    <xacro:include filename="$(find my_robot_urdf)/urdf/arm_coco.xacro" />
     <xacro:include filename="$(find my_robot_urdf)/urdf/arm_yuzi.xacro" />
     <xacro:property name="robot_alex_distance" value="1.8" />
@@ -42,4 +43,5 @@
     <xacro:workbench workbench_name="${workbench_name_2}" workbench_height="${workbench_height_2}" workbench_length="${workbench_length_2}" workbench_width="${workbench_width_2}" />
     <xacro:workbench workbench_name="${workbench_name_3}" workbench_height="${workbench_height_3}" workbench_length="${workbench_length_3}" workbench_width="${workbench_width_3}" />
+    <xacro:my_component component_name="centrifuge_link_1" component_path="package://my_robot_urdf/models/centrifuge.dae"/>
     <!-- Instantiate the centrifuges as the root link -->
     <xacro:centrifuge centrifuge_name="${centrifuge_name_1}" centrifuge_length="${centrifuge_length_1}" centrifuge_diameter="${centrifuge_diameter_1}" />
@@ -76,8 +78,13 @@
         <origin xyz="-${(centrifuge_diameter_1 / 2) + centrifuge_distance_x} ${centrifuge_distance_y} 0" rpy="0 0 0"/>
     </joint>
+    <joint name="base_to_centrifuge_model_1_joint" type="fixed">
+        <parent link="central_base_link"/>
+        <child link="centrifuge_link_1"/>
+        <origin xyz="${(centrifuge_diameter_1 / 2) + centrifuge_distance_x} ${centrifuge_distance_y} ${(centrifuge_length_1) + 0.1879}" rpy="${PI/2} 0 0"/>
+    </joint>
     <!-- Instantiate the arms, attaching it to the central base link -->
     <xacro:arm prefix="alex_" parent_link="central_base_link" xyz="-1 0 ${workbench_height_1}" rpy="0 0 ${PI}" />
     <!-- TODO: Instantiate the arm_coco, attaching it to the central base link -->
-    <!-- <xacro:arm_coco prefix="coco_" parent_link="central_base_link" xyz="0 1 ${workbench_height_1}" rpy="0 0 0" /> -->
+    <xacro:arm_coco prefix="coco_" parent_link="central_base_link" xyz="0 1 ${workbench_height_1}" rpy="0 0 0" />
     <xacro:arm_yuzi prefix="yuzi_" parent_link="central_base_link" xyz="1 0 ${workbench_height_1}" rpy="0 0 0" />
 </robot>

File: ws_robotermodelierung/src/triple_robot_config/config/gazebo_my_robot.urdf (robot description, URDF)
Before this commit: robot my_robot, 30 links, 29 joints
Links:
- removed link alex_arm_link_1
- removed link alex_arm_link_2
- removed link alex_arm_link_3
- removed link alex_arm_link_4
- removed link alex_arm_link_5
- removed link alex_arm_link_6
- removed link alex_base_link
- removed link alex_eef_jaw_1
- removed link alex_eef_jaw_2
- removed link alex_eef_jaw_3
- removed link alex_eef_jaw_4
- removed link alex_eef_link
- removed link coco_eef_link_coco
- added link alex_arm_link_1_alex, mass 26.7048266497369; collision mesh filename=package://my_robot_urdf/meshes/arm_link_1_alex.STL; visual mesh filename=package://my_robot_urdf/meshes/arm_link_1_alex.STL
- added link alex_arm_link_2_alex, mass 14.3270690802686; collision mesh filename=package://my_robot_urdf/meshes/arm_link_2_alex.STL; visual mesh filename=package://my_robot_urdf/meshes/arm_link_2_alex.STL
- added link alex_arm_link_3_alex, mass 27.1450417424437; collision mesh filename=package://my_robot_urdf/meshes/arm_link_3_alex.STL; visual mesh filename=package://my_robot_urdf/meshes/arm_link_3_alex.STL
- added link alex_arm_link_4_alex, mass 9.30858027519608; collision mesh filename=package://my_robot_urdf/meshes/arm_link_4_alex.STL; visual mesh filename=package://my_robot_urdf/meshes/arm_link_4_alex.STL
- added link alex_arm_link_5_alex, mass 0.961734748124672; collision mesh filename=package://my_robot_urdf/meshes/arm_link_5_alex.STL; visual mesh filename=package://my_robot_urdf/meshes/arm_link_5_alex.STL
- added link alex_arm_link_6_alex, mass 0.288779624800079; collision mesh filename=package://my_robot_urdf/meshes/arm_link_6_alex.STL; visual mesh filename=package://my_robot_urdf/meshes/arm_link_6_alex.STL
- added link alex_base_link_alex, mass 33.891578448587; collision mesh filename=package://my_robot_urdf/meshes/base_link_alex.STL; visual mesh filename=package://my_robot_urdf/meshes/base_link_alex.STL
- added link alex_eef_link_alex, mass 1.45406661810263; collision mesh filename=package://my_robot_urdf/meshes/eef_link_alex.STL; visual mesh filename=package://my_robot_urdf/meshes/eef_link_alex.STL
- added link centrifuge_1, mass 500.0; collision cylinder length=0.75 radius=0.5; visual cylinder length=0.75 radius=0.5
- added link centrifuge_2, mass 500.0; collision cylinder length=0.75 radius=0.5; visual cylinder length=0.75 radius=0.5
- added link coco_eef_link_1_coco, mass 0.15332063940157; collision mesh filename=package://my_robot_urdf/meshes/eef_link_1_coco.STL; visual mesh filename=package://my_robot_urdf/meshes/eef_link_1_coco.STL
- added link coco_eef_link_2_coco, mass 0.158859300753402; collision mesh filename=package://my_robot_urdf/meshes/eef_link_2_coco.STL; visual mesh filename=package://my_robot_urdf/meshes/eef_link_2_coco.STL
- added link main_workbench_3, mass 1000.0; collision box size=0.8 5 0.75; visual box size=0.8 5 0.75
- added link yuzi_eef_link_yuzi, mass 0.190738563830904; collision mesh filename=package://my_robot_urdf/meshes/eef_link_yuzi.STL; visual mesh filename=package://my_robot_urdf/meshes/eef_link_yuzi.STL
- link coco_arm_link_3_coco: mass 16.9402164034933 -> 16.1199771168543
- link coco_arm_link_4_coco: mass 7.44374239326319 -> 8.2144132017799
- link coco_arm_link_5_coco: mass 1.52714461517355 -> 1.15468077380916
- link coco_arm_link_6_coco: mass 0.0783717856165202 -> 1.15468077380916
- link main_workbench: geometry collision box size=15 15 0.1; visual box size=15 15 0.1
- link main_workbench_2: geometry collision box size=0.8 5 0.75; visual box size=0.8 5 0.75
- link yuzi_arm_link_3_yuzi: mass 4.48725682214161 -> 4.48725682214162
- link yuzi_arm_link_6_yuzi: mass 0.178247683979378 -> 0.190738563830904
Joints:
- removed joint alex_arm_joint_1
- removed joint alex_arm_joint_2
- removed joint alex_arm_joint_3
- removed joint alex_arm_joint_4
- removed joint alex_arm_joint_5
- removed joint alex_arm_joint_6
- removed joint alex_base_joint
- removed joint alex_eef_jaw_1_joint_fixed
- removed joint alex_eef_jaw_2_joint_fixed
- removed joint alex_eef_jaw_3_joint_fixed
- removed joint alex_eef_jaw_4_joint_fixed
- removed joint alex_eef_link_fixed
- removed joint coco_eef_joint_fixed_coco
- removed joint yuzi_joint_link_1_yuzi
- removed joint yuzi_joint_link_2_yuzi
- removed joint yuzi_joint_link_3_yuzi
- removed joint yuzi_joint_link_4_yuzi
- removed joint yuzi_joint_link_5_yuzi
- removed joint yuzi_joint_link_6_yuzi
- added joint alex_arm_joint_1_alex: type revolute, parent alex_base_link_alex, child alex_arm_link_1_alex, origin xyz=0 0 0.234 rpy=0 0 0, axis 0 0 1, limit lower=-3.1416 upper=3.1416 effort=0 velocity=0
- added joint alex_arm_joint_2_alex: type revolute, parent alex_arm_link_1_alex, child alex_arm_link_2_alex, origin xyz=0.15 -0.1375 0.265 rpy=0 0 0, axis 0 1 0, limit lower=-3.1416 upper=3.1416 effort=0 velocity=0
- added joint alex_arm_joint_3_alex: type revolute, parent alex_arm_link_2_alex, child alex_arm_link_3_alex, origin xyz=0 0 0.7 rpy=0 0 0, axis 0 1 0, limit lower=-3.1416 upper=3.1416 effort=0 velocity=0
- added joint alex_arm_joint_4_alex: type revolute, parent alex_arm_link_3_alex, child alex_arm_link_4_alex, origin xyz=0.29 0.13 0.115 rpy=0 0 0, axis 1 0 0, limit lower=-3.1416 upper=3.1416 effort=0 velocity=0
- added joint alex_arm_joint_5_alex: type revolute, parent alex_arm_link_4_alex, child alex_arm_link_5_alex, origin xyz=0.51 0 0 rpy=0 0 0, axis 0 1 0, limit lower=-3.1416 upper=3.1416 effort=0 velocity=0
- added joint alex_arm_joint_6_alex: type revolute, parent alex_arm_link_5_alex, child alex_arm_link_6_alex, origin xyz=0.045 0 0 rpy=1.5708 0 1.5708, axis 0 0 1, limit lower=-1.5708 upper=4.7124 effort=0 velocity=0
- added joint alex_base_joint_alex: type fixed, parent central_base_link, child alex_base_link_alex, origin xyz=-1 0 0.1 rpy=0 0 3.14159265359
- added joint alex_eef_joint_fixed_alex: type fixed, parent alex_arm_link_6_alex, child alex_eef_link_alex, origin xyz=0 0 0.32173 rpy=0 0 3.1416, axis 0 0 0
- added joint base_to_centrifuge_1_joint: type fixed, parent central_base_link, child centrifuge_1, origin xyz=1.7 1.2 0 rpy=0 0 0
- added joint base_to_centrifuge_2_joint: type fixed, parent central_base_link, child centrifuge_2, origin xyz=-1.7 1.2 0 rpy=0 0 0
- added joint base_to_workbench_3_joint: type fixed, parent central_base_link, child main_workbench_3, origin xyz=-2.2 -2.5 0 rpy=0 0 0
- added joint coco_eef_joint_1_fixed_coco: type fixed, parent coco_arm_link_6_coco, child coco_eef_link_1_coco, origin xyz=0.20975 0.00067738 0.085 rpy=-1.5708 0 -1.5708, axis 0 0 0
- added joint coco_eef_joint_2_fixed_coco: type fixed, parent coco_arm_link_6_coco, child coco_eef_link_2_coco, origin xyz=-0.13985 0.00067738 0.085 rpy=-1.5708 0 1.5708, axis 0 0 0
- added joint yuzi_arm_joint_1_yuzi: type revolute, parent yuzi_base_link_yuzi, child yuzi_arm_link_1_yuzi, origin xyz=0 0 0.274 rpy=0 0 0, axis 0 0 1, limit lower=-3.1416 upper=3.1416 effort=0 velocity=0
- added joint yuzi_arm_joint_2_yuzi: type revolute, parent yuzi_arm_link_1_yuzi, child yuzi_arm_link_2_yuzi, origin xyz=0.15 0 0.29 rpy=-1.5708 0 3.1416, axis 0 0 -1, limit lower=-1.5708 upper=1.5708 effort=0 velocity=0
- added joint yuzi_arm_joint_3_yuzi: type revolute, parent yuzi_arm_link_2_yuzi, child yuzi_arm_link_3_yuzi, origin xyz=0 -0.575 0 rpy=0 0 0, axis 0 0 -1, limit lower=-1.5708 upper=1.5708 effort=0 velocity=0
- added joint yuzi_arm_joint_4_yuzi: type revolute, parent yuzi_arm_link_3_yuzi, child yuzi_arm_link_4_yuzi, origin xyz=-0.1295 -0.04 -0.003 rpy=1.5708 0 -1.5708, axis 0 0 1, limit lower=-3.1416 upper=3.1416 effort=0 velocity=0
- added joint yuzi_arm_joint_5_yuzi: type revolute, parent yuzi_arm_link_4_yuzi, child yuzi_arm_link_5_yuzi, origin xyz=0 0 0.5455 rpy=-1.5708 1.5708 0, axis 0 0 1, limit lower=-1.5708 upper=1.5708 effort=0 velocity=0
- added joint yuzi_arm_joint_6_yuzi: type revolute, parent yuzi_arm_link_5_yuzi, child yuzi_arm_link_6_yuzi, origin xyz=-0.085 0 0 rpy=-1.5708 0 1.5708, axis 0 0 1, limit lower=-3.1416 upper=3.1416 effort=0 velocity=0
- added joint yuzi_eef_joint_fixed_yuzi: type fixed, parent yuzi_arm_link_6_yuzi, child yuzi_eef_link_yuzi, origin xyz=0 0 0.105 rpy=0 -0.031509 0, axis 0 0 0
- joint base_to_workbench_2_joint: origin xyz=2.5 0 0 rpy=0 0 0 -> xyz=2.2 -2.5 0 rpy=0 0 0
- joint coco_arm_joint_6_coco: axis 0 0 1 -> 0 0 -1; origin xyz=0.088678 -0.00048689 -0.0063488 rpy=0 1.5708 0 -> xyz=0.085 0.00067738 -0.0028482 rpy=0 1.5708 0
- joint coco_joint_link_2_coco: origin xyz=-0.14579 0.090292 0.33595 rpy=1.5708 0.12064 -3.1416 -> xyz=0.14579 -0.090292 0.33595 rpy=1.5708 0 0
- joint coco_joint_link_3_coco: origin xyz=0.0017779 0.76236 0 rpy=3.1416 0 2.5562 -> xyz=0.0017779 0.76236 0 rpy=3.1416 0 3.1416
- joint coco_joint_link_4_coco: origin xyz=0.25011 -0.19918 0.073652 rpy=0 1.5708 0 -> xyz=-0.34817 0.19918 0.073652 rpy=3.1416 -1.5708 3.1416
- joint coco_joint_link_5_coco: origin xyz=0 0.0061313 0.60723 rpy=1.5708 -0.32663 -1.5708 -> xyz=0 0.0656 0.50466 rpy=3.1416 -1.5708 0
- joint yuzi_base_joint_yuzi: origin xyz=0 2 0.1 rpy=0 0 0 -> xyz=1 0 0.1 rpy=0 0 0
