Commit message: Implementing three robots

File: ws_robotermodelierung/src/my_robot_urdf/urdf/robot.urdf (robot description, URDF)
Before this commit: robot my_robot, 27 links, 26 joints
Links:
- removed link left_arm_link_1
- removed link left_arm_link_2
- removed link left_arm_link_3
- removed link left_arm_link_4
- removed link left_arm_link_5
- removed link left_arm_link_6
- removed link left_base_link
- removed link left_eef_jaw_1
- removed link left_eef_jaw_2
- removed link left_eef_jaw_3
- removed link left_eef_jaw_4
- removed link left_eef_link
- removed link right_arm_link_1
- removed link right_arm_link_2
- removed link right_arm_link_3
- removed link right_arm_link_4
- removed link right_arm_link_5
- removed link right_arm_link_6
- removed link right_base_link
- removed link right_eef_jaw_1
- removed link right_eef_jaw_2
- removed link right_eef_jaw_3
- removed link right_eef_jaw_4
- removed link right_eef_link
- added link alex_arm_link_1, mass 26.7048266497369; collision mesh filename=package://my_robot_urdf/meshes/arm_link_1.STL; visual mesh filename=package://my_robot_urdf/meshes/arm_link_1.STL
- added link alex_arm_link_2, mass 14.3270690802686; collision mesh filename=package://my_robot_urdf/meshes/arm_link_2.STL; visual mesh filename=package://my_robot_urdf/meshes/arm_link_2.STL
- added link alex_arm_link_3, mass 27.1450417424437; collision mesh filename=package://my_robot_urdf/meshes/arm_link_3.STL; visual mesh filename=package://my_robot_urdf/meshes/arm_link_3.STL
- added link alex_arm_link_4, mass 7.96664349020365; collision mesh filename=package://my_robot_urdf/meshes/arm_link_4.STL; visual mesh filename=package://my_robot_urdf/meshes/arm_link_4.STL
- added link alex_arm_link_5, mass 0.961734748124672; collision mesh filename=package://my_robot_urdf/meshes/arm_link_5.STL; visual mesh filename=package://my_robot_urdf/meshes/arm_link_5.STL
- added link alex_arm_link_6, mass 0.288779624800079; collision mesh filename=package://my_robot_urdf/meshes/arm_link_6.STL; visual mesh filename=package://my_robot_urdf/meshes/arm_link_6.STL
- added link alex_base_link, mass 33.891578448587; collision mesh filename=package://my_robot_urdf/meshes/base_link.STL; visual mesh filename=package://my_robot_urdf/meshes/base_link.STL
- added link alex_eef_jaw_1, mass 0.672155087926634; collision mesh filename=package://my_robot_urdf/meshes/eef_jaw_1.STL; visual mesh filename=package://my_robot_urdf/meshes/eef_jaw_1.STL
- added link alex_eef_jaw_2, mass 0.672155087926635; collision mesh filename=package://my_robot_urdf/meshes/eef_jaw_2.STL; visual mesh filename=package://my_robot_urdf/meshes/eef_jaw_2.STL
- added link alex_eef_jaw_3, mass 0.672155087926635; collision mesh filename=package://my_robot_urdf/meshes/eef_jaw_3.STL; visual mesh filename=package://my_robot_urdf/meshes/eef_jaw_3.STL
- added link alex_eef_jaw_4, mass 0.672155087926635; collision mesh filename=package://my_robot_urdf/meshes/eef_jaw_4.STL; visual mesh filename=package://my_robot_urdf/meshes/eef_jaw_4.STL
- added link alex_eef_link, mass 5.46782575492837; collision mesh filename=package://my_robot_urdf/meshes/eef_link.STL; visual mesh filename=package://my_robot_urdf/meshes/eef_link.STL
- added link coco_arm_link_1_coco, mass 28.7973325809481; collision mesh filename=package://my_robot_urdf/meshes/arm_link_1_coco.STL; visual mesh filename=package://my_robot_urdf/meshes/arm_link_1_coco.STL
- added link coco_arm_link_2_coco, mass 29.9902849835083; collision mesh filename=package://my_robot_urdf/meshes/arm_link_2_coco.STL; visual mesh filename=package://my_robot_urdf/meshes/arm_link_2_coco.STL
- added link coco_arm_link_3_coco, mass 16.9402164034933; collision mesh filename=package://my_robot_urdf/meshes/arm_link_3_coco.STL; visual mesh filename=package://my_robot_urdf/meshes/arm_link_3_coco.STL
- added link coco_arm_link_4_coco, mass 7.44374239326319; collision mesh filename=package://my_robot_urdf/meshes/arm_link_4_coco.STL; visual mesh filename=package://my_robot_urdf/meshes/arm_link_4_coco.STL
- added link coco_arm_link_5_coco, mass 1.52714461517355; collision mesh filename=package://my_robot_urdf/meshes/arm_link_5_coco.STL; visual mesh filename=package://my_robot_urdf/meshes/arm_link_5_coco.STL
- added link coco_arm_link_6_coco, mass 0.0783717856165202; collision mesh filename=package://my_robot_urdf/meshes/arm_link_6_coco.STL; visual mesh filename=package://my_robot_urdf/meshes/arm_link_6_coco.STL
- added link coco_base_link_coco, mass 33.7641312353281; collision mesh filename=package://my_robot_urdf/meshes/base_link_coco.STL; visual mesh filename=package://my_robot_urdf/meshes/base_link_coco.STL
- added link coco_eef_link_coco, mass 0.0881458860458235; collision mesh filename=package://my_robot_urdf/meshes/eef_link_coco.STL; visual mesh filename=package://my_robot_urdf/meshes/eef_link_coco.STL
- added link yuzi_arm_link_1_yuzi, mass 17.6840361237851; collision mesh filename=package://my_robot_urdf/meshes/arm_link_1_yuzi.STL; visual mesh filename=package://my_robot_urdf/meshes/arm_link_1_yuzi.STL
- added link yuzi_arm_link_2_yuzi, mass 21.695061095067; collision mesh filename=package://my_robot_urdf/meshes/arm_link_2_yuzi.STL; visual mesh filename=package://my_robot_urdf/meshes/arm_link_2_yuzi.STL
- added link yuzi_arm_link_3_yuzi, mass 4.48725682214161; collision mesh filename=package://my_robot_urdf/meshes/arm_link_3_yuzi.STL; visual mesh filename=package://my_robot_urdf/meshes/arm_link_3_yuzi.STL
- added link yuzi_arm_link_4_yuzi, mass 7.8906783291211; collision mesh filename=package://my_robot_urdf/meshes/arm_link_4_yuzi.STL; visual mesh filename=package://my_robot_urdf/meshes/arm_link_4_yuzi.STL
- added link yuzi_arm_link_5_yuzi, mass 0.684392926448249; collision mesh filename=package://my_robot_urdf/meshes/arm_link_5_yuzi.STL; visual mesh filename=package://my_robot_urdf/meshes/arm_link_5_yuzi.STL
- added link yuzi_arm_link_6_yuzi, mass 0.178247683979378; collision mesh filename=package://my_robot_urdf/meshes/arm_link_6_yuzi.STL; visual mesh filename=package://my_robot_urdf/meshes/arm_link_6_yuzi.STL
- added link yuzi_base_link_yuzi, mass 13.926198063469; collision mesh filename=package://my_robot_urdf/meshes/base_link_yuzi.STL; visual mesh filename=package://my_robot_urdf/meshes/base_link_yuzi.STL
- link main_workbench: geometry collision box size=2 5 0.1; visual box size=2 5 0.1
- link main_workbench_2: geometry collision box size=2 5 0.6; visual box size=2 5 0.6
Joints:
- removed joint left_arm_joint_1
- removed joint left_arm_joint_2
- removed joint left_arm_joint_3
- removed joint left_arm_joint_4
- removed joint left_arm_joint_5
- removed joint left_arm_joint_6
- removed joint left_base_joint
- removed joint left_eef_jaw_1_joint_fixed
- removed joint left_eef_jaw_2_joint_fixed
- removed joint left_eef_jaw_3_joint_fixed
- removed joint left_eef_jaw_4_joint_fixed
- removed joint left_eef_link_fixed
- removed joint right_arm_joint_1
- removed joint right_arm_joint_2
- removed joint right_arm_joint_3
- removed joint right_arm_joint_4
- removed joint right_arm_joint_5
- removed joint right_arm_joint_6
- removed joint right_base_joint
- removed joint right_eef_jaw_1_joint_fixed
- removed joint right_eef_jaw_2_joint_fixed
- removed joint right_eef_jaw_3_joint_fixed
- removed joint right_eef_jaw_4_joint_fixed
- removed joint right_eef_link_fixed
- added joint alex_arm_joint_1: type revolute, parent alex_base_link, child alex_arm_link_1, origin xyz=0 0 0.234000000000013 rpy=0 0 0, axis 0 0 1, limit lower=-3.1416 upper=3.1416 effort=0 velocity=0
- added joint alex_arm_joint_2: type revolute, parent alex_arm_link_1, child alex_arm_link_2, origin xyz=0.150000000000002 -0.1375 0.265 rpy=1.5707963267949 0 0, axis 0 0 1, limit lower=-3.1416 upper=3.1416 effort=0 velocity=0
- added joint alex_arm_joint_3: type continuous, parent alex_arm_link_2, child alex_arm_link_3, origin xyz=-0.700000000000001 0 0 rpy=3.14159265358979 0 3.14159265358979, axis 0 0 -1, limit lower=-3.1416 upper=3.1416 effort=0 velocity=0
- added joint alex_arm_joint_4: type revolute, parent alex_arm_link_3, child alex_arm_link_4, origin xyz=0.115 0.289996513803296 0.11 rpy=1.5707963267949 0 3.14159265358979, axis 0 0 1, limit lower=-3.1416 upper=3.1416 effort=0 velocity=0
- added joint alex_arm_joint_5: type revolute, parent alex_arm_link_4, child alex_arm_link_5, origin xyz=0 0 0.510003486196704 rpy=1.5707963267949 0 0, axis 0 0 1, limit lower=-4.7124 upper=1.5708 effort=0 velocity=0
- added joint alex_arm_joint_6: type revolute, parent alex_arm_link_5, child alex_arm_link_6, origin xyz=0.0450000000000004 0 0 rpy=-1.5707963267949 0 -1.5707963267949, axis 0 0 1, limit lower=-3.1416 upper=3.1416 effort=0 velocity=0
- added joint alex_base_joint: type fixed, parent central_base_link, child alex_base_link, origin xyz=0 0 0.1 rpy=0 0 0
- added joint alex_eef_jaw_1_joint_fixed: type fixed, parent alex_eef_link, child alex_eef_jaw_1, origin xyz=-0.222284161474005 -0.0199999999999985 -0.0299999999999994 rpy=3.14159265358979 0 0, axis 0 0 0
- added joint alex_eef_jaw_2_joint_fixed: type fixed, parent alex_eef_link, child alex_eef_jaw_2, origin xyz=0.222284161474005 0.0200000000000028 -0.0300000000000008 rpy=0 0 3.14159265358979, axis 0 0 0
- added joint alex_eef_jaw_3_joint_fixed: type fixed, parent alex_eef_link, child alex_eef_jaw_3, origin xyz=0.02 -0.222284161474003 -0.03 rpy=0 0 1.5707963267949, axis 0 0 0
- added joint alex_eef_jaw_4_joint_fixed: type fixed, parent alex_eef_link, child alex_eef_jaw_4, origin xyz=-0.0200000000000002 0.222284161474006 -0.0299999999999999 rpy=0 0 -1.5707963267949, axis 0 0 0
- added joint alex_eef_link_fixed: type fixed, parent alex_arm_link_6, child alex_eef_link, origin xyz=0 0 0.145 rpy=3.14159265358979 0 3.14159265358979, axis 0 0 0
- added joint coco_arm_joint_6_coco: type revolute, parent coco_arm_link_5_coco, child coco_arm_link_6_coco, origin xyz=0.088678 -0.00048689 -0.0063488 rpy=0 1.5708 0, axis 0 0 1, limit lower=-3.1416 upper=3.1416 effort=0 velocity=0
- added joint coco_base_joint_coco: type fixed, parent central_base_link, child coco_base_link_coco, origin xyz=0 1 0.1 rpy=0 0 0
- added joint coco_eef_joint_fixed_coco: type fixed, parent coco_arm_link_6_coco, child coco_eef_link_coco, origin xyz=0 0 0.079322 rpy=0 0 0, axis 0 0 1
- added joint coco_joint_link_1_coco: type revolute, parent coco_base_link_coco, child coco_arm_link_1_coco, origin xyz=0 0 0.18 rpy=0 0 0, axis 0 0 1, limit lower=-3.1416 upper=3.1416 effort=0 velocity=0
- added joint coco_joint_link_2_coco: type revolute, parent coco_arm_link_1_coco, child coco_arm_link_2_coco, origin xyz=-0.14579 0.090292 0.33595 rpy=1.5708 0.12064 -3.1416, axis 0 0 1, limit lower=-3.1416 upper=3.1416 effort=0 velocity=0
- added joint coco_joint_link_3_coco: type revolute, parent coco_arm_link_2_coco, child coco_arm_link_3_coco, origin xyz=0.0017779 0.76236 0 rpy=3.1416 0 2.5562, axis 0 0 -1, limit lower=-3.1416 upper=3.1416 effort=0 velocity=0
- added joint coco_joint_link_4_coco: type revolute, parent coco_arm_link_3_coco, child coco_arm_link_4_coco, origin xyz=0.25011 -0.19918 0.073652 rpy=0 1.5708 0, axis 0 0 1, limit lower=-3.1416 upper=3.1416 effort=0 velocity=0
- added joint coco_joint_link_5_coco: type revolute, parent coco_arm_link_4_coco, child coco_arm_link_5_coco, origin xyz=0 0.0061313 0.60723 rpy=1.5708 -0.32663 -1.5708, axis 0 0 1, limit lower=-3.1416 upper=3.1416 effort=0 velocity=0
- added joint yuzi_base_joint_yuzi: type fixed, parent central_base_link, child yuzi_base_link_yuzi, origin xyz=0 2 0.1 rpy=0 0 0
- added joint yuzi_joint_link_1_yuzi: type revolute, parent yuzi_base_link_yuzi, child yuzi_arm_link_1_yuzi, origin xyz=0 0 0.274 rpy=0 0 0, axis 0 0 1, limit lower=-3.1416 upper=3.1416 effort=0 velocity=0
- added joint yuzi_joint_link_2_yuzi: type revolute, parent yuzi_arm_link_1_yuzi, child yuzi_arm_link_2_yuzi, origin xyz=0.15 0 0.29 rpy=-1.5707963267949 0 3.14159265358979, axis 0 0 -1, limit lower=-1.5708 upper=1.5708 effort=0 velocity=0
- added joint yuzi_joint_link_3_yuzi: type revolute, parent yuzi_arm_link_2_yuzi, child yuzi_arm_link_3_yuzi, origin xyz=0 -0.575 0 rpy=0 0 0, axis 0 0 -1, limit lower=-1.5708 upper=1.5708 effort=0 velocity=0
- added joint yuzi_joint_link_4_yuzi: type revolute, parent yuzi_arm_link_3_yuzi, child yuzi_arm_link_4_yuzi, origin xyz=-0.1295 -0.0399999999999996 -0.00299999999999893 rpy=1.5707963267949 0 -1.5707963267949, axis 0 0 1, limit lower=-3.1416 upper=3.1416 effort=0 velocity=0
- added joint yuzi_joint_link_5_yuzi: type revolute, parent yuzi_arm_link_4_yuzi, child yuzi_arm_link_5_yuzi, origin xyz=0 0 0.5455 rpy=1.5707963267949 1.5707963267949 0, axis 0 0 -1, limit lower=-1.5708 upper=1.5708 effort=0 velocity=0
- added joint yuzi_joint_link_6_yuzi: type revolute, parent yuzi_arm_link_5_yuzi, child yuzi_arm_link_6_yuzi, origin xyz=-0.0850000000000001 0 0 rpy=-1.5707963267949 0 1.5707963267949, axis 0 0 1, limit lower=-3.1416 upper=3.1416 effort=0 velocity=0
- joint base_to_workbench_2_joint: origin xyz=2.0 0 0 rpy=0 0 0 -> xyz=2.5 0 0 rpy=0 0 0

File: ws_robotermodelierung/src/my_robot_urdf/urdf/robot.xacro (robot description, xacro)
@@ -3,12 +3,14 @@
     <xacro:include filename="$(find my_robot_urdf)/urdf/workbench.xacro" />
     <xacro:include filename="$(find my_robot_urdf)/urdf/arm.xacro" />
+    <xacro:include filename="$(find my_robot_urdf)/urdf/arm_coco.xacro" />
+    <xacro:include filename="$(find my_robot_urdf)/urdf/arm_yuzi.xacro" />
     <!-- Define parameters for workbench 1-->
     <xacro:property name="workbench_height_1" value="0.1" />
     <xacro:property name="workbench_length_1" value="2" />
-    <xacro:property name="workbench_width_1" value="4" />
+    <xacro:property name="workbench_width_1" value="5" />
     <xacro:property name="workbench_name_1" value="main_workbench" />
     <xacro:property name="workbench_height_2" value="0.6" />
     <xacro:property name="workbench_length_2" value="2" />
-    <xacro:property name="workbench_width_2" value="4" />
+    <xacro:property name="workbench_width_2" value="5" />
     <xacro:property name="workbench_name_2" value="main_workbench_2" />
     <!-- Instantiate the workbench 1 as the root link -->
@@ -23,13 +25,14 @@
         <parent link="central_base_link"/>
         <child link="${workbench_name_1}"/>
-        <origin xyz="0 0 0" rpy="0 0 0"/> <!-- Adjust this origin as needed -->
+        <origin xyz="0 0 0" rpy="0 0 0"/>
     </joint>
     <joint name="base_to_workbench_2_joint" type="fixed">
         <parent link="central_base_link"/>
         <child link="${workbench_name_2}"/>
-        <origin xyz="${workbench_width_1/2} 0 0" rpy="0 0 0"/> <!-- Adjust this origin as needed -->
+        <origin xyz="${workbench_width_1/2} 0 0" rpy="0 0 0"/>
     </joint>
-    <!-- Instantiate the arm, attaching it to the central base link -->
-    <xacro:arm prefix="left_" parent_link="central_base_link" xyz="0 1 ${workbench_height_1}" rpy="0 0 0" />
-    <xacro:arm prefix="right_" parent_link="central_base_link" xyz="0 -1 ${workbench_height_1}" rpy="0 0 0" />
+    <!-- Instantiate the arms, attaching it to the central base link -->
+    <xacro:arm prefix="alex_" parent_link="central_base_link" xyz="0 0 ${workbench_height_1}" rpy="0 0 0" />
+    <xacro:arm_coco prefix="coco_" parent_link="central_base_link" xyz="0 1 ${workbench_height_1}" rpy="0 0 0" />
+    <xacro:arm_yuzi prefix="yuzi_" parent_link="central_base_link" xyz="0 2 ${workbench_height_1}" rpy="0 0 0" />
 </robot>

Commit message: Add rack and improve layout

File: ws_robotermodelierung/src/my_robot_urdf/urdf/robot.urdf (robot description, URDF)
Before this commit: robot my_robot, 33 links, 32 joints
Links:
- added link main_workbench_4, mass 1000.0; collision box size=1 1 0.75; visual box size=1 1 0.75
- added link rack_link_1, mass 5.0; collision mesh filename=package://my_robot_urdf/models/rack.stl scale=0.001 0.001 0.001; collision mesh filename=package://my_robot_urdf/models/rack.stl scale=0.001 0.001 0.001
- added link rack_link_2, mass 5.0; collision mesh filename=package://my_robot_urdf/models/rack.stl scale=0.001 0.001 0.001; collision mesh filename=package://my_robot_urdf/models/rack.stl scale=0.001 0.001 0.001
- added link rack_link_3, mass 5.0; collision mesh filename=package://my_robot_urdf/models/rack.stl scale=0.001 0.001 0.001; collision mesh filename=package://my_robot_urdf/models/rack.stl scale=0.001 0.001 0.001
Joints:
- added joint base_to_rack_1_joint: type fixed, parent central_base_link, child rack_link_1, origin xyz=2.2 -0.7 0.75 rpy=1.570796326795 0 -1.570796326795
- added joint base_to_rack_2_joint: type fixed, parent central_base_link, child rack_link_2, origin xyz=-2.2 -0.7 0.75 rpy=1.570796326795 0 1.570796326795
- added joint base_to_rack_3_joint: type fixed, parent central_base_link, child rack_link_3, origin xyz=0 2.0 0.75 rpy=1.570796326795 0 0
- added joint base_to_workbench_4_joint: type fixed, parent central_base_link, child main_workbench_4, origin xyz=0 2.0 0 rpy=0 0 0
- joint base_to_centrifuge_1_joint: origin xyz=1.5 1.2 0 rpy=0 0 0 -> xyz=1.3 1.2 0 rpy=0 0 0
- joint base_to_centrifuge_2_joint: origin xyz=-1.5 1.2 0 rpy=0 0 0 -> xyz=-1.3 1.2 0 rpy=0 0 0
- joint base_to_centrifuge_model_1_joint: origin xyz=1.5 1.2 0.9379 rpy=1.570796326795 0 0 -> xyz=1.3 1.2 0.9379 rpy=1.570796326795 0 0
- joint base_to_centrifuge_model_2_joint: origin xyz=-1.5 1.2 0.9379 rpy=1.570796326795 0 0 -> xyz=-1.3 1.2 0.9379 rpy=1.570796326795 0 0

File: ws_robotermodelierung/src/my_robot_urdf/urdf/robot.xacro (robot description, xacro)
@@ -8,4 +8,5 @@
     <xacro:include filename="$(find my_robot_urdf)/urdf/centrifuge.xacro" />
     <xacro:include filename="$(find my_robot_urdf)/urdf/workbench.xacro" />
+    <xacro:include filename="$(find my_robot_urdf)/urdf/rack.xacro" />
     <xacro:include filename="$(find my_robot_urdf)/urdf/arm_coco.xacro" />
     <xacro:include filename="$(find my_robot_urdf)/urdf/arm_yuzi.xacro" />
@@ -31,4 +32,9 @@
     <xacro:property name="workbench_width_3" value="5" />
     <xacro:property name="workbench_name_3" value="main_workbench_3" />
+    <!-- Define parameters for workbench 3-->
+    <xacro:property name="workbench_height_4" value="0.75" />
+    <xacro:property name="workbench_length_4" value="1" />
+    <xacro:property name="workbench_width_4" value="1" />
+    <xacro:property name="workbench_name_4" value="main_workbench_4" />
     <!-- Define parameters for centrifuge 1-->
     <xacro:property name="centrifuge_length_1" value="0.75" />
@@ -45,8 +51,18 @@
     <xacro:property name="centrifuge_model_name_2" value="centrifuge_link_2"/>
     <xacro:property name="centrifuge_2_collada" value="package://my_robot_urdf/models/centrifuge.dae"/>
+    <!-- Define parameters for the rack 2-->
+    <xacro:property name="rack_model_name_1" value="rack_link_1"/>
+    <xacro:property name="rack_model_name_1_stl" value="package://my_robot_urdf/models/rack.stl"/>
+    <!-- Define parameters for the rack 2-->
+    <xacro:property name="rack_model_name_2" value="rack_link_2"/>
+    <xacro:property name="rack_model_name_2_stl" value="package://my_robot_urdf/models/rack.stl"/>
+    <!-- Define parameters for the rack 2-->
+    <xacro:property name="rack_model_name_3" value="rack_link_3"/>
+    <xacro:property name="rack_model_name_3_stl" value="package://my_robot_urdf/models/rack.stl"/>
     <!-- Instantiate the workbenches as the root link -->
     <xacro:workbench_ground workbench_name="${workbench_name_1}" workbench_height="${workbench_height_1}" workbench_length="${workbench_length_1}" workbench_width="${workbench_width_1}" />
     <xacro:workbench workbench_name="${workbench_name_2}" workbench_height="${workbench_height_2}" workbench_length="${workbench_length_2}" workbench_width="${workbench_width_2}" />
     <xacro:workbench workbench_name="${workbench_name_3}" workbench_height="${workbench_height_3}" workbench_length="${workbench_length_3}" workbench_width="${workbench_width_3}" />
+    <xacro:workbench workbench_name="${workbench_name_4}" workbench_height="${workbench_height_4}" workbench_length="${workbench_length_4}" workbench_width="${workbench_width_4}" />
     <!-- Instantiate the centrifuges as the root link -->
     <xacro:centrifuge centrifuge_name="${centrifuge_name_1}" centrifuge_length="${centrifuge_length_1}" centrifuge_diameter="${centrifuge_diameter_1}" />
@@ -54,4 +70,8 @@
     <xacro:centrifuge_model component_name="${centrifuge_model_name_1}" component_path="${centrifuge_1_collada}"/>
     <xacro:centrifuge_model component_name="${centrifuge_model_name_2}" component_path="${centrifuge_2_collada}"/>
+    <!-- Instantiate the racks-->
+    <xacro:rack_model component_name="${rack_model_name_1}" component_path="${rack_model_name_1_stl}" />
+    <xacro:rack_model component_name="${rack_model_name_2}" component_path="${rack_model_name_2_stl}" />
+    <xacro:rack_model component_name="${rack_model_name_3}" component_path="${rack_model_name_3_stl}" />
     <!-- Main body link (central base link) -->
     <link name="central_base_link">
@@ -73,4 +93,9 @@
         <child link="${workbench_name_3}"/>
         <origin xyz="-${(workbench_length_3 / 2) + robot_yuzi_distance} -${workbench_width_3 / 2} 0" rpy="0 0 0"/>
+    </joint>
+    <joint name="base_to_workbench_4_joint" type="fixed">
+        <parent link="central_base_link"/>
+        <child link="${workbench_name_4}"/>
+        <origin xyz="0 ${(workbench_length_4 / 2) + 1.5} 0" rpy="0 0 0"/>
     </joint>
     <!-- Connect each centrifuge to the central base link with a fixed joint -->
@@ -95,4 +120,20 @@
         <origin xyz="-${(centrifuge_diameter_2 / 2) + centrifuge_distance_x} ${centrifuge_distance_y} ${(centrifuge_length_2) + centrifuge_offset}" rpy="${PI/2} 0 0"/>
     </joint>
+    <!-- Connect each rack to the central base link with a fixed joint -->
+    <joint name="base_to_rack_1_joint" type="fixed">
+        <parent link="central_base_link"/>
+        <child link="${rack_model_name_1}"/>
+        <origin xyz="${(workbench_length_2 / 2) + robot_yuzi_distance} ${workbench_length_2 - 1.5} ${workbench_height_2}" rpy="${PI/2} 0 -${PI/2}"/>
+    </joint>
+    <joint name="base_to_rack_2_joint" type="fixed">
+        <parent link="central_base_link"/>
+        <child link="${rack_model_name_2}"/>
+        <origin xyz="-${(workbench_length_3 / 2) + robot_yuzi_distance} ${workbench_length_3 - 1.5} ${workbench_height_3}" rpy="${PI/2} 0 ${PI/2}"/>
+    </joint>
+    <joint name="base_to_rack_3_joint" type="fixed">
+        <parent link="central_base_link"/>
+        <child link="${rack_model_name_3}"/>
+        <origin xyz="0 ${(workbench_length_4 / 2) + 1.5} ${workbench_height_3}" rpy="${PI/2} 0 0"/>
+    </joint>
     <!-- Instantiate the arms, attaching it to the central base link -->
     <xacro:arm prefix="alex_" parent_link="central_base_link" xyz="-1 0 ${workbench_height_1}" rpy="0 0 ${PI}" />
