Commit message: Add pose script

File: ws_robotermodelierung/src/triple_robot_config/config/gazebo_my_robot.urdf (robot description, URDF)
Before this commit: robot my_robot, 31 links, 30 joints
Links:
- added link centrifuge_link_1, mass 1.0; collision mesh filename=package://my_robot_urdf/models/centrifuge.dae scale=1 1 1; visual mesh filename=package://my_robot_urdf/models/centrifuge.dae scale=1 1 1
- added link centrifuge_link_2, mass 1.0; collision mesh filename=package://my_robot_urdf/models/centrifuge.dae scale=1 1 1; visual mesh filename=package://my_robot_urdf/models/centrifuge.dae scale=1 1 1
- link centrifuge_1: geometry collision cylinder length=0.75 radius=0.3; visual cylinder length=0.75 radius=0.3
- link centrifuge_2: geometry collision cylinder length=0.75 radius=0.3; visual cylinder length=0.75 radius=0.3
Joints:
- added joint base_to_centrifuge_model_1_joint: type fixed, parent central_base_link, child centrifuge_link_1, origin xyz=1.5 1.2 0.9379 rpy=1.570796326795 0 0
- added joint base_to_centrifuge_model_2_joint: type fixed, parent central_base_link, child centrifuge_link_2, origin xyz=-1.5 1.2 0.9379 rpy=1.570796326795 0 0
- joint base_to_centrifuge_1_joint: origin xyz=1.7 1.2 0 rpy=0 0 0 -> xyz=1.5 1.2 0 rpy=0 0 0
- joint base_to_centrifuge_2_joint: origin xyz=-1.7 1.2 0 rpy=0 0 0 -> xyz=-1.5 1.2 0 rpy=0 0 0
